Commit message: Finished restructuring code

File: franka_sim/assets/fr3.urdf (robot description, URDF)
Before this commit: robot fr3, 22 links, 21 joints
Links:
- added link fr3_hand, mass 0.6544; collision mesh filename=meshes/robot_ee/franka_hand_white/collision/hand.stl; visual mesh filename=meshes/robot_ee/franka_hand_white/visual/hand.dae
- added link fr3_hand_tcp
- added link fr3_leftfinger, mass 0.0291; collision box size=17.5e-3 15.2e-3 18.5e-3; collision box size=17.5e-3 7e-3 23.5e-3
- added link fr3_rightfinger, mass 0.0291; collision box size=17.5e-3 15.2e-3 18.5e-3; collision box size=17.5e-3 7e-3 23.5e-3
- link fr3_link0: geometry collision mesh filename=meshes/robots/fr3/collision/link0.stl; visual mesh filename=meshes/robots/fr3/visual/link0.dae
- link fr3_link1: geometry collision mesh filename=meshes/robots/fr3/collision/link1.stl; visual mesh filename=meshes/robots/fr3/visual/link1.dae
- link fr3_link2: geometry collision mesh filename=meshes/robots/fr3/collision/link2.stl; visual mesh filename=meshes/robots/fr3/visual/link2.dae
- link fr3_link3: geometry collision mesh filename=meshes/robots/fr3/collision/link3.stl; visual mesh filename=meshes/robots/fr3/visual/link3.dae
- link fr3_link4: geometry collision mesh filename=meshes/robots/fr3/collision/link4.stl; visual mesh filename=meshes/robots/fr3/visual/link4.dae
- link fr3_link5: geometry collision mesh filename=meshes/robots/fr3/collision/link5.stl; visual mesh filename=meshes/robots/fr3/visual/link5.dae
- link fr3_link6: geometry collision mesh filename=meshes/robots/fr3/collision/link6.stl; visual mesh filename=meshes/robots/fr3/visual/link6.dae
- link fr3_link7: geometry collision mesh filename=meshes/robots/fr3/collision/link7.stl; visual mesh filename=meshes/robots/fr3/visual/link7.dae
Joints:
- added joint fr3_finger_joint1: type prismatic, parent fr3_hand, child fr3_leftfinger, origin xyz=0 0 0.0584 rpy=0 0 0, axis 0 1 0, limit lower=0.0 upper=0.04 effort=100 velocity=0.2
- added joint fr3_finger_joint2: type prismatic, parent fr3_hand, child fr3_rightfinger, origin xyz=0 0 0.0584 rpy=0 0 3.141592653589793, axis 0 1 0, limit lower=0.0 upper=0.04 effort=100 velocity=0.2, mimic joint=fr3_finger_joint1
- added joint fr3_hand_joint: type fixed, parent fr3_link8, child fr3_hand, origin xyz=0 0 0 rpy=0 0 -0.7853981633974483
- added joint fr3_hand_tcp_joint: type fixed, parent fr3_hand, child fr3_hand_tcp, origin xyz=0 0 0.1034 rpy=0 0 0

Commit message: Restructured assets directory and removed unused files

File: franka_sim/assets/fr3.urdf (robot description, URDF)
Before this commit: robot fr3, 26 links, 25 joints
Links:
- link fr3_hand: geometry collision mesh filename=meshes/hand_coll.stl; visual mesh filename=meshes/hand_vis.dae
- link fr3_leftfinger: geometry collision box size=17.5e-3 15.2e-3 18.5e-3; collision box size=17.5e-3 7e-3 23.5e-3
- link fr3_link0: geometry collision mesh filename=meshes/link0_coll.stl; visual mesh filename=meshes/link0_vis.dae
- link fr3_link1: geometry collision mesh filename=meshes/link1_coll.stl; visual mesh filename=meshes/link1_vis.dae
- link fr3_link2: geometry collision mesh filename=meshes/link2_coll.stl; visual mesh filename=meshes/link2_vis.dae
- link fr3_link3: geometry collision mesh filename=meshes/link3_coll.stl; visual mesh filename=meshes/link3_vis.dae
- link fr3_link4: geometry collision mesh filename=meshes/link4_coll.stl; visual mesh filename=meshes/link4_vis.dae
- link fr3_link5: geometry collision mesh filename=meshes/link5_coll.stl; visual mesh filename=meshes/link5_vis.dae
- link fr3_link6: geometry collision mesh filename=meshes/link6_coll.stl; visual mesh filename=meshes/link6_vis.dae
- link fr3_link7: geometry collision mesh filename=meshes/link7_coll.stl; visual mesh filename=meshes/link7_vis.dae
- link fr3_rightfinger: geometry collision box size=17.5e-3 15.2e-3 18.5e-3; collision box size=17.5e-3 7e-3 23.5e-3
