Commit message: Corrected URDF provided by GetModelCommand

File: franky_sim/assets/fr3_clean.urdf (robot description, URDF)
Before this commit: robot fr3, 22 links, 21 joints
Links:
- removed link fr3_link0
- removed link fr3_link0_accelerometer_bottom
- removed link fr3_link0_accelerometer_top
- removed link fr3_link1
- removed link fr3_link1_accelerometer_bottom
- removed link fr3_link1_accelerometer_top
- removed link fr3_link2
- removed link fr3_link2_accelerometer_bottom
- removed link fr3_link2_accelerometer_top
- removed link fr3_link3
- removed link fr3_link3_accelerometer_bottom
- removed link fr3_link3_accelerometer_top
- removed link fr3_link4
- removed link fr3_link4_accelerometer_bottom
- removed link fr3_link4_accelerometer_top
- removed link fr3_link5
- removed link fr3_link5_accelerometer_bottom
- removed link fr3_link5_accelerometer_top
- removed link fr3_link6
- removed link fr3_link7
- removed link fr3_link8
- added link link0, mass 2.3966
- added link link0_accelerometer_bottom
- added link link0_accelerometer_top
- added link link1, mass 2.9274653454
- added link link1_accelerometer_bottom
- added link link1_accelerometer_top
- added link link2, mass 2.9355370338
- added link link2_accelerometer_bottom
- added link link2_accelerometer_top
- added link link3, mass 2.2449013699
- added link link3_accelerometer_bottom
- added link link3_accelerometer_top
- added link link4, mass 2.6155955791
- added link link4_accelerometer_bottom
- added link link4_accelerometer_top
- added link link5, mass 2.3271207594
- added link link5_accelerometer_bottom
- added link link5_accelerometer_top
- added link link6, mass 1.8170376524
- added link link7, mass 0.6271432862
- added link link8
Joints:
- removed joint fr3_base_joint
- removed joint fr3_joint1
- removed joint fr3_joint2
- removed joint fr3_joint3
- removed joint fr3_joint4
- removed joint fr3_joint5
- removed joint fr3_joint6
- removed joint fr3_joint7
- removed joint fr3_joint8
- removed joint fr3_link0_accelerometer_bottom_joint
- removed joint fr3_link0_accelerometer_top_joint
- removed joint fr3_link1_accelerometer_bottom_joint
- removed joint fr3_link1_accelerometer_top_joint
- removed joint fr3_link2_accelerometer_bottom_joint
- removed joint fr3_link2_accelerometer_top_joint
- removed joint fr3_link3_accelerometer_bottom_joint
- removed joint fr3_link3_accelerometer_top_joint
- removed joint fr3_link4_accelerometer_bottom_joint
- removed joint fr3_link4_accelerometer_top_joint
- removed joint fr3_link5_accelerometer_bottom_joint
- removed joint fr3_link5_accelerometer_top_joint
- added joint base_joint: type fixed, parent base, child link0, origin xyz=0 0 0 rpy=0 0 0
- added joint joint1: type revolute, parent link0, child link1, origin xyz=0 0 0.333 rpy=0 0 0, axis 0 0 1, limit lower=-2.9007 upper=2.9007 effort=87.0 velocity=2.62
- added joint joint2: type revolute, parent link1, child link2, origin xyz=0 0 0 rpy=-1.570796326794897 0 0, axis 0 0 1, limit lower=-1.8361 upper=1.8361 effort=87.0 velocity=2.62
- added joint joint3: type revolute, parent link2, child link3, origin xyz=0 -0.316 0 rpy=1.570796326794897 0 0, axis 0 0 1, limit lower=-2.9007 upper=2.9007 effort=87.0 velocity=2.62
- added joint joint4: type revolute, parent link3, child link4, origin xyz=0.0825 0 0 rpy=1.570796326794897 0 0, axis 0 0 1, limit lower=-3.077 upper=-0.1169 effort=87.0 velocity=2.62
- added joint joint5: type revolute, parent link4, child link5, origin xyz=-0.0825 0.384 0 rpy=-1.570796326794897 0 0, axis 0 0 1, limit lower=-2.8763 upper=2.8763 effort=12.0 velocity=5.26
- added joint joint6: type revolute, parent link5, child link6, origin xyz=0 0 0 rpy=1.570796326794897 0 0, axis 0 0 1, limit lower=0.4398 upper=4.6216 effort=12.0 velocity=4.18
- added joint joint7: type revolute, parent link6, child link7, origin xyz=0.088 0 0 rpy=1.570796326794897 0 0, axis 0 0 1, limit lower=-3.0508 upper=3.0508 effort=12.0 velocity=5.26
- added joint joint8: type fixed, parent link7, child link8, origin xyz=0 0 0.107 rpy=0 0 0
- added joint link0_accelerometer_bottom_joint: type fixed, parent link0, child link0_accelerometer_bottom, origin xyz=-0.019739 0.0015506 0.05075 rpy=0.0 0.0 -1.5708
- added joint link0_accelerometer_top_joint: type fixed, parent link0, child link0_accelerometer_top, origin xyz=-0.017402 -0.007872 0.04715 rpy=3.1416 0.0 0.0
- added joint link1_accelerometer_bottom_joint: type fixed, parent link1, child link1_accelerometer_bottom, origin xyz=0.01974 -0.08975 0.00155 rpy=-1.5708 1.5708 0.0
- added joint link1_accelerometer_top_joint: type fixed, parent link1, child link1_accelerometer_top, origin xyz=0.017402 -0.093352 -0.00787 rpy=-1.5708 0.0 3.1416
- added joint link2_accelerometer_bottom_joint: type fixed, parent link2, child link2_accelerometer_bottom, origin xyz=0.019737 -0.11875 -0.00155 rpy=1.5708 -1.5708 0.0
- added joint link2_accelerometer_top_joint: type fixed, parent link2, child link2_accelerometer_top, origin xyz=0.017403 -0.11715 0.00787 rpy=1.5708 0.0 3.1416
- added joint link3_accelerometer_bottom_joint: type fixed, parent link3, child link3_accelerometer_bottom, origin xyz=0.062769 0.073756 0.00155 rpy=1.5708 1.5708 0.0
- added joint link3_accelerometer_top_joint: type fixed, parent link3, child link3_accelerometer_top, origin xyz=0.065099 0.077352 -0.00787 rpy=-1.5708 0.0 0.0
- added joint link4_accelerometer_bottom_joint: type fixed, parent link4, child link4_accelerometer_bottom, origin xyz=-0.062775 0.049753 0.00155 rpy=-1.5708 1.5708 0.0
- added joint link4_accelerometer_top_joint: type fixed, parent link4, child link4_accelerometer_top, origin xyz=-0.0651 0.046252 -0.00787 rpy=-1.5708 0.0 -3.1416
- added joint link5_accelerometer_bottom_joint: type fixed, parent link5, child link5_accelerometer_bottom, origin xyz=-0.019742 0.082275 0.00146 rpy=1.5708 1.5708 0.0
- added joint link5_accelerometer_top_joint: type fixed, parent link5, child link5_accelerometer_top, origin xyz=-0.017363 0.085872 -0.00795 rpy=-1.5708 0.0 0.0
